File: Kick/808.kicad_pcb (KiCad board)
At the start: 2 copper layers, 109.9 x 62.2 mm, 57 parts, among them J1 Trigger In, J2 Trigger OUT, Q1 BC546, Q2 BC546, Q3 BC556, Q4 BC546, Q5 BC546, Q6 BC546, SW1 Trigger, U1 TL072

Commit message: kick done with higher track width
Parts:
- added J3: CONN, Connectors_Terminal_Blocks:TerminalBlock_bornier-3_P5.08mm, F.Cu at (52.7, 97.8)
Routing:
- net -15V: track 73.9 -> 138.3 mm, vias 0 -> 1
- net GND: track 263.9 -> 311.1 mm
- net +15V: track 180.2 -> 191.1 mm
- net Net-(C13-Pad1): track 11.4 -> 15.2 mm
- net Net-(C11-Pad1): track 0.00 -> 3.18 mm
- net Net-(R20-Pad1): track 89.5 -> 87.6 mm
- net Net-(C12-Pad2): track 74.7 -> 75.5 mm
Other:
- net class Default: trace_width 0.25 -> 0.5
